File: HeartRateMonitor.kicad_sch (KiCad schematic)
At the start: 64 parts, among them J1 USB_C_Receptacle_USB2.0, J2 SWD, J3 Conn_01x08_Pin, U1 CH340E, U11 LM2904, U2 LM2904, U3 TLV62130, U4 STM32G030F6Px, U5 TPS60403, U6 LM2904, U9 AD5272BCP

Commit message: finalize hardware
Parts:
- removed C13: 15uF, Capacitor_SMD:C_0402_1005Metric, symbol Device:C_Small
- removed R10, R11, R12, R6, R7, R9: 0, Resistor_SMD:R_0603_1608Metric, symbol Device:R_Small
- removed R15: 4K87, Resistor_SMD:R_0603_1608Metric, symbol Device:R_Small
- C12: value 22uF -> 10uF; footprint Capacitor_SMD:C_0805_2012Metric -> Capacitor_SMD:C_0603_1608Metric
- C21: value 82uF -> 33uF; footprint Capacitor_SMD:C_0603_1608Metric -> Capacitor_SMD:C_1206_3216Metric
- C22: value 68uF -> 15uF; footprint Capacitor_SMD:C_0603_1608Metric -> Capacitor_SMD:C_0402_1005Metric
- J1: footprint FP:TYPE-C-31-M-31 -> FP:TYPE-C-SMD_HX-TYPE-C-16PIN
- R14: value 12K -> 15K8
- R25: value 22K6 -> 15K8
- R26: value 442 -> 3K92
- U11, U2, U6: footprint (none) -> Package_SO:VSSOP-8_3.0x3.0mm_P0.65mm
Connections:
- net SCR_CS: now also J3.7 (Pin_7)
- net SCR_DC: now also J3.5 (Pin_5)
- net SCR_RES: now also J3.6 (Pin_6)
- net at C12.2: now also R14.1, U2.3 (+)
- no-connect marks 8 -> 9

Commit message: Hardware Cleanup
Connections:
- net HIGH_NPH: now reaches R16.1, R26.2, U2.6 (-), U2.7
Other:
- note added: "HighPass Filter - 2 level Butterwurth"
- note added: "LowPass Filter - For HR Calculating"
- note added: "LowPass Filter - For Wave Displaying"
- note added: "Main Microcontroller & SWD Debug"
- note added: "Passband 1Hz Stopband 0.4Hz Attenuation -40dB"
- note added: "Passband 4Hz Stopband 6Hz Attenuation -20dB"
- note added: "Passband 6Hz Stopband 10Hz Attenuation -30dB"
- note added: "Photodiode & Transimpedance Amplifier"
- note added: "Programmable Gain Amplifier"
- note added: "Screen Connector"
- note added: "System 3V3 Power"
- note added: "System Negative Voltage Source"
- note added: "USB C Power UART Debug and Config"
- note removed: "我把这幅杰作留在这 因为我看了半天怎么想也没想明白为啥要把这个电容放在这里 光电二极管的信号频率不高的 在输入脚串电容不就开路了吗？想要有人帮忙指点一下"
- note removed: "鉴定为困傻了（"
- company: (none) -> Yao Haizhou
- title: (none) -> HeartRateMonitor
- moved on the sheet: C10, C11, C12, C14, C15, C16, C17, C18, C19, C20, C21, C22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
